Commit message: obj resized

File: kuka_lego_sorter/resources/urdf/bar_blue.urdf (robot description, URDF)
Before this commit: robot bar, 1 links, 0 joints
Links:
- link base: mass 1.0 -> 0.1

File: kuka_lego_sorter/resources/urdf/bar_green.urdf (robot description, URDF)
Before this commit: robot lego_1_3, 1 links, 0 joints
Links:
- link base: geometry collision mesh filename=OBJ/bar.obj scale=1 1 1; visual mesh filename=OBJ/bar.obj scale=1 1 1

File: kuka_lego_sorter/resources/urdf/bar_red.urdf (robot description, URDF)
Before this commit: robot bar, 1 links, 0 joints
Links:
- link base: mass 1.0 -> 0.1

File: kuka_lego_sorter/resources/urdf/bar_yellow.urdf (robot description, URDF)
Before this commit: robot bar, 1 links, 0 joints
Links:
- link base: mass 1.0 -> 0.1

File: kuka_lego_sorter/resources/urdf/corn_blue.urdf (robot description, URDF)
Before this commit: robot corn, 1 links, 0 joints
Links:
- link base: mass 1.0 -> 0.1

File: kuka_lego_sorter/resources/urdf/corn_green.urdf (robot description, URDF)
Before this commit: robot lego_1_3, 1 links, 0 joints
Links:
- link base: geometry collision mesh filename=OBJ/corn.obj scale=1 1 1; visual mesh filename=OBJ/corn.obj scale=1 1 1

File: kuka_lego_sorter/resources/urdf/corn_red.urdf (robot description, URDF)
Before this commit: robot corn, 1 links, 0 joints
Links:
- link base: mass 1.0 -> 0.1

File: kuka_lego_sorter/resources/urdf/corn_yellow.urdf (robot description, URDF)
Before this commit: robot corn, 1 links, 0 joints
Links:
- link base: mass 1.0 -> 0.1

File: kuka_lego_sorter/resources/urdf/lego_1_1_blue.urdf (robot description, URDF)
Before this commit: robot lego_1_1, 1 links, 0 joints
Links:
- link base: mass 1.0 -> 0.1

File: kuka_lego_sorter/resources/urdf/lego_1_1_green.urdf (robot description, URDF)
Before this commit: robot lego_1_1, 1 links, 0 joints
Links:
- link base: mass 1.0 -> 0.1

File: kuka_lego_sorter/resources/urdf/lego_1_1_orange.urdf (robot description, URDF)
Before this commit: robot lego_1_1, 1 links, 0 joints
Links:
- link base: mass 1.0 -> 0.1

File: kuka_lego_sorter/resources/urdf/lego_1_1_purple.urdf (robot description, URDF)
Before this commit: robot lego_1_1, 1 links, 0 joints
Links:
- link base: mass 1.0 -> 0.1

File: kuka_lego_sorter/resources/urdf/lego_1_1_red.urdf (robot description, URDF)
Before this commit: robot lego_1_1, 1 links, 0 joints
Links:
- link base: mass 1.0 -> 0.1

File: kuka_lego_sorter/resources/urdf/lego_1_1_skyblue.urdf (robot description, URDF)
Before this commit: robot lego_1_1, 1 links, 0 joints
Links:
- link base: mass 1.0 -> 0.1

File: kuka_lego_sorter/resources/urdf/lego_1_1_yellow.urdf (robot description, URDF)
Before this commit: robot lego_1_1, 1 links, 0 joints
Links:
- link base: mass 1.0 -> 0.1

File: kuka_lego_sorter/resources/urdf/lego_1_2_blue.urdf (robot description, URDF)
Before this commit: robot lego_1_2, 1 links, 0 joints
Links:
- link base: mass 1.0 -> 0.1

File: kuka_lego_sorter/resources/urdf/lego_1_2_green.urdf (robot description, URDF)
Before this commit: robot lego_1_2, 1 links, 0 joints
Links:
- link base: mass 1.0 -> 0.1

File: kuka_lego_sorter/resources/urdf/lego_1_2_orange.urdf (robot description, URDF)
Before this commit: robot lego_1_2, 1 links, 0 joints
Links:
- link base: mass 1.0 -> 0.1

File: kuka_lego_sorter/resources/urdf/lego_1_2_purple.urdf (robot description, URDF)
Before this commit: robot lego_1_2, 1 links, 0 joints
Links:
- link base: mass 1.0 -> 0.1

File: kuka_lego_sorter/resources/urdf/lego_1_2_red.urdf (robot description, URDF)
Before this commit: robot lego_1_2, 1 links, 0 joints
Links:
- link base: mass 1.0 -> 0.1
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